File: vhdci2dp.kicad_pcb (KiCad board)
At the start: 4 copper layers, 45 x 61 mm, 64 parts, among them J1 MiniDP, J2 71430-015, J3 MiniDP, J4 MiniDP, J5 MiniDP

Commit message: revA
Parts:
- added REF**: stitch, vhdci2dp:stitch_16_12, F.Cu at (171.6, 92.6)
- added REF**: stitch, vhdci2dp:stitch_16_12, F.Cu at (175.3, 83.4)
- added REF**: stitch, vhdci2dp:stitch_16_12, F.Cu at (166.2, 85.0)
- added REF**: stitch, vhdci2dp:stitch_16_12, F.Cu at (169.5, 85.0)
- added REF**: stitch, vhdci2dp:stitch_16_12, F.Cu at (169.5, 82.8)
- added REF**: stitch, vhdci2dp:stitch_16_12, F.Cu at (166.2, 83.0)
- added REF**: stitch, vhdci2dp:stitch_16_12, F.Cu at (166.2, 81.1)
- added REF**: stitch, vhdci2dp:stitch_16_12, F.Cu at (169.8, 79.2)
- added REF**: stitch, vhdci2dp:stitch_16_12, F.Cu at (165.5, 79.2)
- added REF**: stitch, vhdci2dp:stitch_16_12, F.Cu at (173.0, 50.2)
- added REF**: stitch, vhdci2dp:stitch_16_12, F.Cu at (176.4, 53.5)
- added REF**: stitch, vhdci2dp:stitch_16_12, F.Cu at (166.9, 97.2)
- added REF**: stitch, vhdci2dp:stitch_16_12, F.Cu at (165.2, 55.1)
- added REF**: stitch, vhdci2dp:stitch_16_12, F.Cu at (168.2, 56.5)
- added REF**: stitch, vhdci2dp:stitch_16_12, F.Cu at (171.6, 59.9)
- added REF**: stitch, vhdci2dp:stitch_16_12, F.Cu at (174.8, 62.9)
- added REF**: stitch, vhdci2dp:stitch_16_12, F.Cu at (172.1, 58.2)
- added REF**: stitch, vhdci2dp:stitch_16_12, F.Cu at (169.4, 55.5)
- added REF**: stitch, vhdci2dp:stitch_16_12, F.Cu at (166.5, 52.8)
- added REF**: stitch, vhdci2dp:stitch_16_12, F.Cu at (165.9, 50.5)
- added REF**: stitch, vhdci2dp:stitch_16_12, F.Cu at (168.7, 51.1)
- added REF**: stitch, vhdci2dp:stitch_16_12, F.Cu at (170.6, 53.1)
- added REF**: stitch, vhdci2dp:stitch_16_12, F.Cu at (177.6, 97.8)
- added REF**: stitch, vhdci2dp:stitch_16_12, F.Cu at (173.0, 55.3)
- added REF**: stitch, vhdci2dp:stitch_16_12, F.Cu at (174.9, 57.1)
- added REF**: stitch, vhdci2dp:stitch_16_12, F.Cu at (177.5, 59.8)
- added REF**: stitch, vhdci2dp:stitch_16_12, F.Cu at (167.5, 87.1)
- added REF**: stitch, vhdci2dp:stitch_16_12, F.Cu at (165.0, 87.1)
- added REF**: stitch, vhdci2dp:stitch_16_12, F.Cu at (163.5, 91.8)
- added REF**: stitch, vhdci2dp:stitch_16_12, F.Cu at (165.4, 91.8)
- added REF**: stitch, vhdci2dp:stitch_16_12, F.Cu at (165.4, 95.5)
- added REF**: stitch, vhdci2dp:stitch_16_12, F.Cu at (168.5, 92.8)
- added REF**: stitch, vhdci2dp:stitch_16_12, F.Cu at (178.9, 88.3)
- added REF**: stitch, vhdci2dp:stitch_16_12, F.Cu at (177.6, 98.5)
- added REF**: stitch, vhdci2dp:stitch_16_12, F.Cu at (178.9, 83.4)
- added REF**: stitch, vhdci2dp:stitch_16_12, F.Cu at (178.9, 78.2)
- added REF**: stitch, vhdci2dp:stitch_16_12, F.Cu at (173.2, 79.2)
- added REF**: stitch, vhdci2dp:stitch_16_12, F.Cu at (167.3, 61.9)
- added REF**: stitch, vhdci2dp:stitch_16_12, F.Cu at (165.4, 61.9)
- added REF**: stitch, vhdci2dp:stitch_16_12, F.Cu at (163.3, 61.9)
- added REF**: stitch, vhdci2dp:stitch_16_12, F.Cu at (161.2, 61.9)
- added REF**: stitch, vhdci2dp:stitch_16_12, F.Cu at (168.0, 72.3)
- added REF**: stitch, vhdci2dp:stitch_16_12, F.Cu at (165.9, 72.3)
- added REF**: stitch, vhdci2dp:stitch_16_12, F.Cu at (168.0, 70.0)
- added REF**: stitch, vhdci2dp:stitch_16_12, F.Cu at (177.6, 99.2)
- added REF**: stitch, vhdci2dp:stitch_16_12, F.Cu at (165.9, 70.0)
- added REF**: stitch, vhdci2dp:stitch_16_12, F.Cu at (164.3, 70.0)
- added REF**: stitch, vhdci2dp:stitch_16_12, F.Cu at (163.5, 72.3)
- added REF**: stitch, vhdci2dp:stitch_16_12, F.Cu at (177.6, 70.9)
- added REF**: stitch, vhdci2dp:stitch_16_12, F.Cu at (175.9, 69.6)
- added REF**: stitch, vhdci2dp:stitch_16_12, F.Cu at (177.7, 66.1)
- added REF**: stitch, vhdci2dp:stitch_16_12, F.Cu at (172.7, 67.8)
- added REF**: stitch, vhdci2dp:stitch_16_12, F.Cu at (170.1, 67.8)
- added REF**: stitch, vhdci2dp:stitch_16_12, F.Cu at (167.6, 67.8)
- added REF**: stitch, vhdci2dp:stitch_16_12, F.Cu at (165.1, 67.8)
- added REF**: stitch, vhdci2dp:stitch_16_12, F.Cu at (177.7, 50.7)
- added REF**: stitch, vhdci2dp:stitch_16_12, F.Cu at (168.3, 66.0)
- added REF**: stitch, vhdci2dp:stitch_16_12, F.Cu at (166.1, 66.0)
- added REF**: stitch, vhdci2dp:stitch_16_12, F.Cu at (164.0, 66.0)
- added REF**: stitch, vhdci2dp:stitch_16_12, F.Cu at (175.3, 61.2)
- added REF**: stitch, vhdci2dp:stitch_16_12, F.Cu at (177.4, 63.9)
- added REF**: stitch, vhdci2dp:stitch_16_12, F.Cu at (178.9, 60.8)
- added REF**: stitch, vhdci2dp:stitch_16_12, F.Cu at (178.9, 57.9)
- added REF**: stitch, vhdci2dp:stitch_16_12, F.Cu at (167.4, 48.1)
- added REF**: stitch, vhdci2dp:stitch_16_12, F.Cu at (166.1, 48.1)
- added REF**: stitch, vhdci2dp:stitch_16_12, F.Cu at (164.8, 48.1)
- added REF**: stitch, vhdci2dp:stitch_16_12, F.Cu at (177.7, 49.2)
- added REF**: stitch, vhdci2dp:stitch_16_12, F.Cu at (163.6, 48.1)
- added REF**: stitch, vhdci2dp:stitch_16_12, F.Cu at (168.1, 46.6)
- added REF**: stitch, vhdci2dp:stitch_16_12, F.Cu at (167.0, 46.6)
- added REF**: stitch, vhdci2dp:stitch_16_12, F.Cu at (166.0, 46.6)
- added REF**: stitch, vhdci2dp:stitch_16_12, F.Cu at (164.7, 46.6)
- added REF**: stitch, vhdci2dp:stitch_16_12, F.Cu at (163.6, 46.6)
- added REF**: stitch, vhdci2dp:stitch_16_12, F.Cu at (162.6, 46.6)
- added REF**: stitch, vhdci2dp:stitch_16_12, F.Cu at (177.7, 50.0)
- added REF**: stitch, vhdci2dp:stitch_16_12, F.Cu at (174.1, 82.5)
Other:
- board size 45 x 61 mm -> 43 x 61 mm
